Commit message: Prametrized configration

File: LAB_2/urdf/rotating.urdf.xacro (robot description, xacro)
@@ -15,4 +15,5 @@
 				<cylinder length="0.6" radius="0.2" />
 			</geometry>
+			<origin xyz="0 0 -0.3" rpy="0 0 0" />
 		</visual>
 	</link>

Commit message: Upgraded graphics and parametrization

File: LAB_2/urdf/rotating.urdf.xacro (robot description, xacro)
@@ -13,7 +13,7 @@
 		<visual>
 			<geometry>
-				<cylinder length="0.6" radius="0.2" />
+				<cylinder length="${params['a1']}" radius="0.2" />
 			</geometry>
-			<origin xyz="0 0 -0.3" rpy="0 0 0" />
+			<origin xyz="${.5*params['a1']} 0 0" rpy="0 1.57 0" />
 		</visual>
 	</link>
@@ -21,6 +21,7 @@
 		<visual>
 			<geometry>
-				<cylinder length="0.6" radius="0.2" />
+				<cylinder length="${params['a2']}" radius="0.2" />
 			</geometry>
+			<origin xyz="${.5*params['a1']} 0 0" rpy="0 1.57 0" />
 		</visual>
 	</link>
@@ -35,5 +36,5 @@
 		<parent link="base" />
 		<child link="link1" />
-		<origin xyz="${params['joint1']['pos']}" rpy="${params['joint1']['rpy']}" />
+		<origin xyz="0 0 0" rpy="${params['joint1-rpy']}" />
 		<axis xyz="0 0 1" />
 	</joint>
@@ -41,12 +42,13 @@
 		<parent link="link1" />
 		<child link="link2" />
-		<origin xyz="${params['joint2']['pos']}" rpy="${params['joint2']['rpy']}" />
+		<origin xyz="${params['a1']} 0 0" rpy="${params['joint2-rpy']}" />
 		<axis xyz="0 0 1" />
 	</joint>
-	<joint name="joint3" type="continuous">
+	<joint name="joint3" type="prismatic">
 		<parent link="link2" />
 		<child link="manip" />
-		<origin xyz="${params['joint3']['pos']}" rpy="${params['joint3']['rpy']}" />
+		<origin xyz="${params['a2']} 0 0" rpy="${params['joint3-rpy']}" />
 		<axis xyz="0 0 1" />
+		<limit effort="5" velocity="5" lower="${-params['d3']}" upper="${params['d3']}" />
 	</joint>
 </robot>
