Commit message: Small fixes

File: LAB_2/urdf/fixed.urdf.xacro (robot description, xacro)
@@ -13,6 +13,7 @@
 		<visual>
 			<geometry>
-				<cylinder length="0.6" radius="0.2" />
+				<cylinder length="${params['a1']}" radius="0.2" />
 			</geometry>
+			<origin xyz="${.5*params['a1']} 0 0" rpy="0 1.57 0" />
 		</visual>
 	</link>
@@ -20,6 +21,7 @@
 		<visual>
 			<geometry>
-				<cylinder length="0.6" radius="0.2" />
+				<cylinder length="${params['a2']}" radius="0.2" />
 			</geometry>
+			<origin xyz="${.5*params['a2']} 0 0" rpy="0 1.57 0" />
 		</visual>
 	</link>
@@ -34,15 +36,15 @@
 		<parent link="base" />
 		<child link="link1" />
-		<origin xyz="${params['joint1']['pos']}" rpy="${params['joint1']['rpy']}" />
+		<origin xyz="0 0 0" rpy="${params['joint1-rpy']}" />
 	</joint>
 	<joint name="joint2" type="fixed">
 		<parent link="link1" />
 		<child link="link2" />
-		<origin xyz="${params['joint2']['pos']}" rpy="${params['joint2']['rpy']}" />
+		<origin xyz="${params['a1']} 0 0" rpy="${params['joint2-rpy']}" />
 	</joint>
 	<joint name="joint3" type="fixed">
 		<parent link="link2" />
 		<child link="manip" />
-		<origin xyz="${params['joint3']['pos']}" rpy="${params['joint3']['rpy']}" />
+		<origin xyz="${params['a2']} 0 ${params['d3']}" rpy="${params['joint3-rpy']}" />
 	</joint>
 </robot>

File: LAB_2/urdf/rotating.urdf.xacro (robot description, xacro)
@@ -23,5 +23,5 @@
 				<cylinder length="${params['a2']}" radius="0.2" />
 			</geometry>
-			<origin xyz="${.5*params['a1']} 0 0" rpy="0 1.57 0" />
+			<origin xyz="${.5*params['a2']} 0 0" rpy="0 1.57 0" />
 		</visual>
 	</link>

Commit message: Final fixes+ static launch

File: LAB_2/urdf/fixed.urdf.xacro (robot description, xacro)
@@ -29,6 +29,7 @@
 		<visual>
 			<geometry>
-				<cylinder length="0.3" radius="0.1" />
+				<cylinder length="${params['d3']}" radius="0.1" />
 			</geometry>
+			<origin xyz="0 0 ${-.5*params['d3']}" rpy="0 0 0" />
 		</visual>
 	</link>
@@ -36,15 +37,15 @@
 		<parent link="base" />
 		<child link="link1" />
-		<origin xyz="0 0 0" rpy="${params['joint1-rpy']}" />
+		<origin xyz="${params['joint1']['pos']}" rpy="${params['joint1']['rpy']}" />
 	</joint>
 	<joint name="joint2" type="fixed">
 		<parent link="link1" />
 		<child link="link2" />
-		<origin xyz="${params['a1']} 0 0" rpy="${params['joint2-rpy']}" />
+		<origin xyz="${params['joint2']['pos']}" rpy="${params['joint2']['rpy']}" />
 	</joint>
 	<joint name="joint3" type="fixed">
 		<parent link="link2" />
 		<child link="manip" />
-		<origin xyz="${params['a2']} 0 ${params['d3']}" rpy="${params['joint3-rpy']}" />
+		<origin xyz="${params['joint3']['pos']}" rpy="${params['joint3']['rpy']}" />
 	</joint>
 </robot>

File: LAB_2/urdf/rotating.urdf.xacro (robot description, xacro)
@@ -29,6 +29,7 @@
 		<visual>
 			<geometry>
-				<cylinder length="0.3" radius="0.1" />
+				<cylinder length="${params['d3']}" radius="0.1" />
 			</geometry>
+			<origin xyz="0 0 ${-.5*params['d3']}" rpy="0 0 0" />
 		</visual>
 	</link>
@@ -36,5 +37,5 @@
 		<parent link="base" />
 		<child link="link1" />
-		<origin xyz="0 0 0" rpy="${params['joint1-rpy']}" />
+		<origin xyz="${params['joint1']['pos']}" rpy="${params['joint1']['rpy']}" />
 		<axis xyz="0 0 1" />
 	</joint>
@@ -42,5 +43,5 @@
 		<parent link="link1" />
 		<child link="link2" />
-		<origin xyz="${params['a1']} 0 0" rpy="${params['joint2-rpy']}" />
+		<origin xyz="${params['joint2']['pos']}" rpy="${params['joint2']['rpy']}" />
 		<axis xyz="0 0 1" />
 	</joint>
@@ -48,7 +49,7 @@
 		<parent link="link2" />
 		<child link="manip" />
-		<origin xyz="${params['a2']} 0 0" rpy="${params['joint3-rpy']}" />
+		<origin xyz="${params['joint3']['pos']}" rpy="${params['joint3']['rpy']}" />
 		<axis xyz="0 0 1" />
-		<limit effort="5" velocity="5" lower="${-params['d3']}" upper="${params['d3']}" />
+		<limit effort="5" velocity="5" lower="${-params['d3']}" upper="0" />
 	</joint>
 </robot>
